Commit message: Changed params, seems really nice + added move_demo from luna

File: gobot_simulation/gobot_description/urdf/gobot.urdf.xacro (robot description, xacro)
@@ -30,5 +30,5 @@
     <xacro:property name="lower_base_height" value="0.068" />
     <xacro:property name="base_space_height" value="0.022" />
-    <xacro:property name="base_space_width" value="0.2" />
+    <xacro:property name="base_space_width" value="0.25" />
     <!-- Laser -->
     <xacro:property name="laser_width" value="0.01" />
@@ -80,5 +80,5 @@
     <caster_wheel fb="back" lr="left" parent="base_link" translateX="${-(base_width/2 - 0.080)}" translateY="${base_length/2 - 0.110}" translateZ="${-(lower_base_height / 2 - 0.037) + 0.008}" flipY="1"/>
     <!-- Hokuyo Laser -->
-    <hokuyo_04lx_laser name="hokuyo" parent="base_link" ros_topic="/scan" update_rate="20" min_angle="${-pi/2}" max_angle="${pi/2}" translateX="${base_width/2 - 0.058}" translateY="0" translateZ="${-0.01 + originZ}" visualize="1"/>
+    <hokuyo_04lx_laser name="hokuyo" parent="base_link" ros_topic="/scan" update_rate="20" min_angle="${-2.094395102}" max_angle="${2.094395102}" translateX="${base_width/2 - 0.04266}" translateY="0" translateZ="${-0.01 + originZ}" visualize="1"/>
     <!-- Cliff sensor, IR technology on real robot but we use a sonar here to simulate -->
     <!-- In order; front left, back left, front right, back right -->

Commit message: New local planner : teb_local_planner, still needs some tuning

File: gobot_simulation/gobot_description/urdf/gobot.urdf.xacro (robot description, xacro)
@@ -28,6 +28,6 @@
     <xacro:property name="base_length" value="0.599" />
     <xacro:property name="base_height" value="0.185" />
-    <xacro:property name="lower_base_height" value="0.068" />
-    <xacro:property name="base_space_height" value="0.022" />
+    <xacro:property name="lower_base_height" value="0.04" />
+    <xacro:property name="base_space_height" value="0.05" />
     <xacro:property name="base_space_width" value="0.25" />
     <!-- Laser -->
@@ -102,5 +102,5 @@
     <sonar_sensor name="prox_right" parent="base_link" ros_topic="/sensors/sonar_sensor/proximity_right" update_rate="20" min_range="0.05" max_range="0.15" field_of_view="0.05" ray_count="1" pos_x="${-base_width/2}" pos_y="-0.085" pos_z="0.15" rotation_z="${pi}" gaussian_noise="0.0" resolution="0.01" visualize="1"/>
     <!-- Battery sensors -->
-    <battery name="left_battery" parent="base_link" height="${battery_height}" radius="${battery_radius}" translateX="${-base_width/2 + 0.08}" translateY="0.049" translateZ="0.025" rotationX="${pi/2}" collision="left_battery_collision" update_rate="20"/>
-    <battery name="right_battery" parent="base_link" height="${battery_height}" radius="${battery_radius}" translateX="${-base_width/2 + 0.08}" translateY="-0.049" translateZ="0.025" rotationX="${pi/2}" collision="right_battery_collision" update_rate="20"/>
+    <battery name="left_battery" parent="base_link" height="${battery_height}" radius="${battery_radius}" translateX="${-base_width/2 + 0.08}" translateY="0.049" translateZ="0.040" rotationX="${pi/2}" collision="left_battery_collision" update_rate="20"/>
+    <battery name="right_battery" parent="base_link" height="${battery_height}" radius="${battery_radius}" translateX="${-base_width/2 + 0.08}" translateY="-0.049" translateZ="0.040" rotationX="${pi/2}" collision="right_battery_collision" update_rate="20"/>
 </robot>

Commit message: modification for new version gobot

File: gobot_simulation/gobot_description/urdf/gobot.urdf.xacro (robot description, xacro)
@@ -25,6 +25,6 @@
     <xacro:include filename="$(find gobot_description)/urdf/battery/battery.urdf.xacro" />
     <!-- Base -->
-    <xacro:property name="base_width" value="0.648" />
-    <xacro:property name="base_length" value="0.599" />
+    <xacro:property name="base_width" value="0.50" />
+    <xacro:property name="base_length" value="0.550" />
     <xacro:property name="base_height" value="0.185" />
     <xacro:property name="lower_base_height" value="0.04" />

Commit message: modified simulation

File: gobot_simulation/gobot_description/urdf/gobot.urdf.xacro (robot description, xacro)
@@ -25,6 +25,6 @@
     <xacro:include filename="$(find gobot_description)/urdf/battery/battery.urdf.xacro" />
     <!-- Base -->
-    <xacro:property name="base_width" value="0.50" />
-    <xacro:property name="base_length" value="0.550" />
+    <xacro:property name="base_width" value="0.648" />
+    <xacro:property name="base_length" value="0.599" />
     <xacro:property name="base_height" value="0.185" />
     <xacro:property name="lower_base_height" value="0.04" />
@@ -80,17 +80,17 @@
     <caster_wheel fb="back" lr="left" parent="base_link" translateX="${-(base_width/2 - 0.080)}" translateY="${base_length/2 - 0.110}" translateZ="${-(lower_base_height / 2 - 0.037) + 0.008}" flipY="1"/>
     <!-- Hokuyo Laser -->
-    <hokuyo_04lx_laser name="hokuyo" parent="base_link" ros_topic="/scan" update_rate="20" min_angle="${-2.094395102}" max_angle="${2.094395102}" translateX="${base_width/2 - 0.04266}" translateY="0" translateZ="0.25" visualize="1"/>
+    <hokuyo_04lx_laser name="hokuyo" parent="base_link" ros_topic="/scan" update_rate="20" min_angle="${-2.094395102}" max_angle="${2.094395102}" translateX="${base_width/2 - 0.04266}" translateY="0" translateZ="${-0.01 + originZ}" visualize="1"/>
     <!-- Cliff sensor, IR technology on real robot but we use a sonar here to simulate -->
     <!-- In order; front left, back left, front right, back right -->
-    <cliff_sensor name="cliff_sensor" parent="base_link" ros_topic="cliff_sensor_topic" update_rate="10" min_range="0.03" max_range="2.0" field_of_view="0.05" ray_count="1" pos_x="${base_width/2-0.02}" pos_y="${-(base_width/2 - 0.10)}" pos_z="0.05" rotation_y="${pi/2}" gaussian_noise="0.03" resolution="0.01" />
-    <cliff_sensor name="cliff_sensor_2" parent="base_link" ros_topic="cliff_sensor_2_topic" update_rate="10" min_range="0.01" max_range="2.0" field_of_view="0.05" ray_count="1" pos_x="${-base_width/2+0.02}" pos_y="${-(base_width/2 - 0.10)}" pos_z="0.05" rotation_y="${pi/2}" gaussian_noise="0.03" resolution="0.01" />
-    <cliff_sensor name="cliff_sensor_3" parent="base_link" ros_topic="cliff_sensor_3_topic" update_rate="10" min_range="0.01" max_range="2.0" field_of_view="0.05" ray_count="1" pos_x="${base_width/2-0.02}" pos_y="${(base_width/2 - 0.10)}" pos_z="0.05" rotation_y="${pi/2}" gaussian_noise="0.03" resolution="0.01" />
-    <cliff_sensor name="cliff_sensor_4" parent="base_link" ros_topic="cliff_sensor_4_topic" update_rate="10" min_range="0.01" max_range="2.0" field_of_view="0.05" ray_count="1" pos_x="${-base_width/2+0.02}" pos_y="${(base_width/2 - 0.10)}" pos_z="0.05" rotation_y="${pi/2}" gaussian_noise="0.03" resolution="0.01" />
+    <cliff_sensor name="cliff_sensor" parent="base_link" ros_topic="cliff_sensor_topic" update_rate="10" min_range="0.03" max_range="2.0" field_of_view="0.05" ray_count="1" pos_x="${base_width/2-0.02}" pos_y="${-(base_width/2 - 0.10)}" pos_z="${originZ - lower_base_height/2}" rotation_y="${pi/2}" gaussian_noise="0.03" resolution="0.01" />
+    <cliff_sensor name="cliff_sensor_2" parent="base_link" ros_topic="cliff_sensor_2_topic" update_rate="10" min_range="0.01" max_range="2.0" field_of_view="0.05" ray_count="1" pos_x="${-base_width/2+0.02}" pos_y="${-(base_width/2 - 0.10)}" pos_z="${originZ - lower_base_height/2}" rotation_y="${pi/2}" gaussian_noise="0.03" resolution="0.01" />
+    <cliff_sensor name="cliff_sensor_3" parent="base_link" ros_topic="cliff_sensor_3_topic" update_rate="10" min_range="0.01" max_range="2.0" field_of_view="0.05" ray_count="1" pos_x="${base_width/2-0.02}" pos_y="${(base_width/2 - 0.10)}" pos_z="${originZ - lower_base_height/2}" rotation_y="${pi/2}" gaussian_noise="0.03" resolution="0.01" />
+    <cliff_sensor name="cliff_sensor_4" parent="base_link" ros_topic="cliff_sensor_4_topic" update_rate="10" min_range="0.01" max_range="2.0" field_of_view="0.05" ray_count="1" pos_x="${-base_width/2+0.02}" pos_y="${(base_width/2 - 0.10)}" pos_z="${originZ - lower_base_height/2}" rotation_y="${pi/2}" gaussian_noise="0.03" resolution="0.01" />
     <!-- Sonar sensors, in order: rear, left side, right side, front right and front left -->
-    <sonar_sensor name="sonar_rear" parent="base_link" ros_topic="/sensors/sonar_sensor/sonar_rear" update_rate="20" min_range="0.15" max_range="2.5" field_of_view="${pi/18}" ray_count="10" pos_x="${-base_width/2}" pos_y="-0.065"  pos_z="0.38" rotation_z="${pi}" gaussian_noise="0.01" resolution="0.0174" visualize="${visualize}"/>
-    <sonar_sensor name="sonar_left" parent="base_link" ros_topic="/sensors/sonar_sensor/sonar_left" update_rate="20" min_range="0.15" max_range="2.5" field_of_view="${pi/18}" ray_count="10" pos_x="-0.009" pos_y="${base_length/2}" pos_z="0.388" rotation_z="${pi/2}" gaussian_noise="0.01" resolution="0.0174" visualize="${visualize}"/>
-    <sonar_sensor name="sonar_right" parent="base_link" ros_topic="/sensors/sonar_sensor/sonar_right" update_rate="20" min_range="0.15" max_range="2.5" field_of_view="${pi/18}" ray_count="10" pos_x="-0.009" pos_y="${-base_length/2}" pos_z="0.388" rotation_z="${3*pi/2}" gaussian_noise="0.01" resolution="0.0174" visualize="${visualize}"/>
-    <sonar_sensor name="sonar_front_right" parent="base_link" ros_topic="/sensors/sonar_sensor/sonar_front_right" update_rate="20" min_range="0.15" max_range="2.5" field_of_view="${pi/18}" ray_count="10" pos_x="${base_width/2}" pos_y="-0.070" pos_z="0.328" rotation_z="0.0" gaussian_noise="0.01" resolution="0.0174" visualize="${visualize}"/>
-    <sonar_sensor name="sonar_front_left" parent="base_link" ros_topic="/sensors/sonar_sensor/sonar_front_left" update_rate="20" min_range="0.15" max_range="2.5" field_of_view="${pi/18}" ray_count="10" pos_x="${base_width/2}" pos_y="0.070" pos_z="0.328" rotation_z="0.0" gaussian_noise="0.01" resolution="0.0174" visualize="${visualize}"/>
+    <sonar_sensor name="sonar_rear" parent="base_link" ros_topic="/sensors/sonar_sensor/sonar_rear" update_rate="20" min_range="0.15" max_range="2.5" field_of_view="${pi/18}" ray_count="10" pos_x="${-base_width/2}" pos_y="-0.065"  pos_z="0.08" rotation_z="${pi}" gaussian_noise="0.01" resolution="0.0174" visualize="${visualize}"/>
+    <sonar_sensor name="sonar_left" parent="base_link" ros_topic="/sensors/sonar_sensor/sonar_left" update_rate="20" min_range="0.15" max_range="2.5" field_of_view="${pi/18}" ray_count="10" pos_x="-0.009" pos_y="${base_length/2}" pos_z="0.088" rotation_z="${pi/2}" gaussian_noise="0.01" resolution="0.0174" visualize="${visualize}"/>
+    <sonar_sensor name="sonar_right" parent="base_link" ros_topic="/sensors/sonar_sensor/sonar_right" update_rate="20" min_range="0.15" max_range="2.5" field_of_view="${pi/18}" ray_count="10" pos_x="-0.009" pos_y="${-base_length/2}" pos_z="0.088" rotation_z="${3*pi/2}" gaussian_noise="0.01" resolution="0.0174" visualize="${visualize}"/>
+    <sonar_sensor name="sonar_front_right" parent="base_link" ros_topic="/sensors/sonar_sensor/sonar_front_right" update_rate="20" min_range="0.15" max_range="2.5" field_of_view="${pi/18}" ray_count="10" pos_x="${base_width/2}" pos_y="-0.070" pos_z="0.128" rotation_z="0.0" gaussian_noise="0.01" resolution="0.0174" visualize="${visualize}"/>
+    <sonar_sensor name="sonar_front_left" parent="base_link" ros_topic="/sensors/sonar_sensor/sonar_front_left" update_rate="20" min_range="0.15" max_range="2.5" field_of_view="${pi/18}" ray_count="10" pos_x="${base_width/2}" pos_y="0.070" pos_z="0.128" rotation_z="0.0" gaussian_noise="0.01" resolution="0.0174" visualize="${visualize}"/>
     <!-- IR sensors -->
     <camera_sensor name="rear" parent="base_link" pos_x="${-base_width/2}" pos_y="0" pos_z="0.126" rotation_z="0" angle="${pi * 15 / 180}"/>
